Commit message: Fix the detection problem to avoid chasing a non-white ball

File: catkin_ws/src/my_robot/urdf/my_robot.xacro (robot description, xacro)
@@ -62,5 +62,4 @@
         <cylinder length="0.05" radius="0.1"/>
       </geometry>
-      <material name="orange"/>
     </visual>
     <inertial>
@@ -82,5 +81,4 @@
         <cylinder length="0.05" radius="0.1"/>
       </geometry>
-      <material name="orange"/>
     </visual>
     <inertial>
@@ -166,9 +164,3 @@
     <axis xyz="0 1 0"/>
   </joint>
-   <gazebo reference="right_wheel">
-      <material>Gazebo/Blue</material>
-   </gazebo>
-   <gazebo reference="left_wheel">
-      <material>Gazebo/Blue</material>
-   </gazebo>
 </robot>
